File: hw/sch_pcb/USTSIPIN02A.kicad_sch (KiCad schematic)
At the start: 66 parts, among them M1 HOLE, M2 HOLE, M3 HOLE, M4 HOLE, M5 BMI-S-210-F, M6 BMI-S-210-F, M7 BMI-S-210-F, M8 BMI-S-204-F, Q1 2SK2394-6, U1 OPA2314, U2 OPA2314, U3 ISL21080DIH312Z-TK 1V25, U4 TS7211, U5 TS5A4594

Commit message: Edit schema
Parts:
- C17, C3: value 4u7 -> 1uF
Changed lines of the file:
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@@
       (effects (font (size 1.27 1.27)) (justify left))
     )
-    (property "Value" "4u7" (id 1) (at 47.371 133.223 0)
+    (property "Value" "1uF" (id 1) (at 47.371 133.223 0)
       (effects (font (size 1.27 1.27)) (justify left))
     )
@@
       (effects (font (size 1.27 1.27)) (justify left))
     )
-    (property "Value" "4u7" (id 1) (at 145.161 137.033 0)
+    (property "Value" "1uF" (id 1) (at 145.161 137.033 0)
       (effects (font (size 1.27 1.27)) (justify left))
     )
@@
       (reference "#PWR?") (unit 1) (value "GND") (footprint "")
     )
+    (path "/00000000-0000-0000-0000-00005c4aedd8/69adadb9-ff3c-4ce2-814d-b306f29ff7c0"
+      (reference "#PWR?") (unit 1) (value "GND") (footprint "")
+    )
     (path "/00000000-0000-0000-0000-00005c4aedd8/dc503e7a-3881-44c7-9dce-fab3105d1bb4"
       (reference "BT?") (unit 1) (value "KEYS2998") (footprint "")
@@
     )
     (path "/00000000-0000-0000-0000-00005b39c727"
-      (reference "C3") (unit 1) (value "4u7") (footprint "Capacitor_SMD:C_0603_1608Metric")
+      (reference "C3") (unit 1) (value "1uF") (footprint "Capacitor_SMD:C_0603_1608Metric")
     )
     (path "/00000000-0000-0000-0000-00005b46aed9"
@@
     )
     (path "/00000000-0000-0000-0000-00005b3e1723"
-      (reference "C17") (unit 1) (value "4u7") (footprint "Capacitor_SMD:C_0603_1608Metric")
+      (reference "C17") (unit 1) (value "1uF") (footprint "Capacitor_SMD:C_0603_1608Metric")
     )
     (path "/00000000-0000-0000-0000-00005b3e8e3e"
@@
       (reference "C59") (unit 1) (value "100nF") (footprint "Capacitor_SMD:C_0603_1608Metric")
     )
+    (path "/00000000-0000-0000-0000-00005c4aedd8/5c120615-7b34-4376-98c4-994ae5b3b131"
+      (reference "C?") (unit 1) (value "100nF") (footprint "Capacitor_SMD:C_0603_1608Metric")
+    )
     (path "/00000000-0000-0000-0000-00005c69bcb4/b879c0f5-5e6c-4b4f-bb4c-6b0f2760c9ee"

Commit message: Editing PCB and schema
Parts:
- removed M5, M6, M7: BMI-S-210-F, Mlab_Mechanical:BMI-S-210-F, symbol MLAB_MECHANICAL:HOLE
- C1, C21, C23, C4, C55, C56, C57, C58, C6, C7, C8, C9: value 10uF -> (none); footprint Capacitor_SMD:C_0603_1608Metric -> (none)
- C10, C11, C12, C13, C14, C16, C2, C20, C59: value 100nF -> (none); footprint Capacitor_SMD:C_0603_1608Metric -> (none)
- C15: value 3n3 -> (none); footprint Capacitor_SMD:C_0603_1608Metric -> (none)
- C17, C24, C3, C37: value 1uF -> (none); footprint Capacitor_SMD:C_0603_1608Metric -> (none)
- C18: value 2n2 -> (none); footprint Capacitor_SMD:C_0603_1608Metric -> (none)
- C19: value 1nF/NP0 -> (none); footprint Capacitor_SMD:C_0805_2012Metric -> (none)
- C5: value 1pFNP0 251R15S1R0AV4E -> (none); footprint Capacitor_SMD:C_0805_2012Metric -> (none)
- C53: value 10uF -> (none); footprint Resistor_SMD:R_0603_1608Metric -> (none)
- D2: value S2744-09 -> (none); footprint Mlab_D:HAMAMATSU_S2744-09 -> (none)
- M1, M2, M3, M4: value HOLE -> (none); footprint Mlab_Mechanical:MountingHole_3mm -> (none)
- M8: value BMI-S-204-F -> (none); footprint RF_Shielding:Laird_Technologies_BMI-S-204-F_32.00x32.00mm -> (none)
- Q1: value 2SK2394-6 -> (none); footprint Package_TO_SOT_SMD:SOT-23 -> (none)
- R1: value 10R -> (none); footprint Resistor_SMD:R_0603_1608Metric -> (none)
- R10, R8: value 1k -> (none); footprint Resistor_SMD:R_0603_1608Metric -> (none)
- R11, R14, R15, R16, R19, R22, R9: value 4k7 -> (none); footprint Resistor_SMD:R_0603_1608Metric -> (none)
- R12, R7: value 10k -> (none); footprint Resistor_SMD:R_0603_1608Metric -> (none)
- R13: value 2k2 -> (none); footprint Resistor_SMD:R_0603_1608Metric -> (none)
- R2, R3, R4, R40, R5: value 470R -> (none); footprint Resistor_SMD:R_0603_1608Metric -> (none)
- R39: value 100R -> (none); footprint Resistor_SMD:R_0603_1608Metric -> (none)
- R41: value 0R -> (none); footprint Resistor_SMD:R_0603_1608Metric -> (none)
- R6: value 10M -> (none); footprint Resistor_SMD:R_0603_1608Metric -> (none)
- U1, U2: value OPA2314 -> (none); footprint Package_SO:SOIC-8_3.9x4.9mm_P1.27mm -> (none)
- U3: value ISL21080DIH312Z-TK 1V25 -> (none); footprint Package_TO_SOT_SMD:SOT-23 -> (none)
- U4: value TS7211 -> (none); footprint Package_TO_SOT_SMD:SOT-23-5_HandSoldering -> (none)
- U5: value TS5A4594 -> (none); footprint Package_TO_SOT_SMD:SOT-23-5_HandSoldering -> (none)
Other:
- moved on the sheet: M1, M2, M3, M4, M8

Commit message: Edit PCB
Parts:
- C1, C21, C23, C4, C55, C56, C57, C58, C6, C7, C8, C9: value (none) -> 10uF; footprint (none) -> Capacitor_SMD:C_0603_1608Metric
- C10, C11, C12, C13, C14, C16, C2, C20, C59: value (none) -> 100nF; footprint (none) -> Capacitor_SMD:C_0603_1608Metric
- C15: value (none) -> 3n3; footprint (none) -> Capacitor_SMD:C_0603_1608Metric
- C17, C24, C3, C37: value (none) -> 1uF; footprint (none) -> Capacitor_SMD:C_0603_1608Metric
- C18: value (none) -> 2n2; footprint (none) -> Capacitor_SMD:C_0603_1608Metric
- C19: value (none) -> 1nF/NP0; footprint (none) -> Capacitor_SMD:C_0805_2012Metric
- C5: value (none) -> 1pFNP0 251R15S1R0AV4E; footprint (none) -> Capacitor_SMD:C_0805_2012Metric
- C53: value (none) -> 10uF; footprint (none) -> Resistor_SMD:R_0603_1608Metric
- D2: value (none) -> S2744-09; footprint (none) -> Mlab_D:HAMAMATSU_S2744-09
- M1, M2, M3, M4: value (none) -> HOLE; footprint (none) -> Mlab_Mechanical:MountingHole_3mm
- M8: value (none) -> BMI-S-204-F; footprint (none) -> RF_Shielding:Laird_Technologies_BMI-S-204-F_32.00x32.00mm
- Q1: value (none) -> 2SK2394-6; footprint (none) -> Package_TO_SOT_SMD:SOT-23
- R1: value (none) -> 10R; footprint (none) -> Resistor_SMD:R_0603_1608Metric
- R10, R8: value (none) -> 1k; footprint (none) -> Resistor_SMD:R_0603_1608Metric
- R11, R14, R15, R16, R19, R22, R9: value (none) -> 4k7; footprint (none) -> Resistor_SMD:R_0603_1608Metric
- R12, R7: value (none) -> 10k; footprint (none) -> Resistor_SMD:R_0603_1608Metric
- R13: value (none) -> 2k2; footprint (none) -> Resistor_SMD:R_0603_1608Metric
- R2, R3, R4, R40, R5: value (none) -> 470R; footprint (none) -> Resistor_SMD:R_0603_1608Metric
- R39: value (none) -> 100R; footprint (none) -> Resistor_SMD:R_0603_1608Metric
- R41: value (none) -> 0R; footprint (none) -> Resistor_SMD:R_0603_1608Metric
- R6: value (none) -> 10M; footprint (none) -> Resistor_SMD:R_0603_1608Metric
- U1, U2: value (none) -> OPA2314; footprint (none) -> Package_SO:SOIC-8_3.9x4.9mm_P1.27mm
- U3: value (none) -> ISL21080DIH312Z-TK 1V25; footprint (none) -> Package_TO_SOT_SMD:SOT-23
- U4: value (none) -> TS7211; footprint (none) -> Package_TO_SOT_SMD:SOT-23-5_HandSoldering
- U5: value (none) -> TS5A4594; footprint (none) -> Package_TO_SOT_SMD:SOT-23-5_HandSoldering

Commit message: uprava stranky, submodul
Other:
- company: Mlab www.mlab.cz -> UST.cz
- title: NAME -> USTSIPIN02A
Changed lines of the file:
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@@
   (paper "A4")
   (title_block
-    (title "NAME")
-    (date "%F")
-    (rev "REV")
-    (company "Mlab www.mlab.cz")
-    (comment 1 "VERSION")
-    (comment 2 "Short description \\nTwo lines are maximum")
-    (comment 3 "nickname <email@example.com>")
-    (comment 4 "BSD")
+    (title "USTSIPIN02A")
+    (date "2022-05-22")
+    (company "UST.cz")
+    (comment 2 "USTSIPIN, Silicon PIN dosimeter")
+    (comment 3 "info@ust.cz")
   )
   (junction (at 96.52 36.83) (diameter 1.016) (color 0 0 0 0)
