File: hw/sch_pcb/USTSIPIN02A.kicad_pcb (KiCad board)
At the start: 4 copper layers, 90.9 x 50.3 mm, 154 parts, among them J1 SM08B-GHS-TB, J2 SD_Card-FPS009-4200-0, J22 HEADER_2x03, J3 SM06B-GHS-TB, J4 USBC_USB4105-GF-A, J5 HEADER_1x01, J6 HEADER_1x01, J7 SM03B-GHS-TB, M1 HOLE, M2 HOLE, M3 HOLE, M4 HOLE, M8 BMI-S-204-F, Q1 2SK2394-6, Q2 BC817-25, Q3 BC817-25, Q4 BC817-25, U1 OPA2314, U10 ATMEGA1284P-AU, U11 PCF85263A, U12 MIC5504-3.3YM5, U2 OPA2314, U3 ISL21080DIH312Z-TK 1V25, U4 TS7211, U5 TS5A4594, U6 AT24CS64-SSHM, U7 USBLC6-2SC6, U8 TPS613222ADBV, U9 FT231XQ, Y1 16MHz, Y2 ABS07-120-32.768KHZ-T

Commit message: Update PCB from schematics.
Parts:
- R3: value 470R -> 10R
- R45: value 100R -> 10R
- Y1: value 16MHz -> 8 MHz

Commit message: Schematics structure change.
Connections:
- net /A renamed /sensor/A
- net /K renamed /sensor/K
- net /Ubiasout renamed /sensor/Ubiasout
- net /power/D+ renamed /USB interface/D+
- net /power/D- renamed /USB interface/D-
- net /power/DM renamed /USB interface/DM
- net /power/DP renamed /USB interface/DP
- net /power/RXLED/CBUS1 renamed /USB interface/RXLED/CBUS1
- net /power/TXLED/CBUS2 renamed /USB interface/TXLED/CBUS2
- C11 pad 1: /VCC1 -> /power/VCC1
- C12 pad 1: /VCC2 -> /power/VCC2
- C13 pad 1: /VCC3 -> /power/VCC3
- C14 pad 1: /VCC4 -> /power/VCC4
- C53 pad 1: /VCC5 -> /power/VCC5
- C59 pad 1: /VCC5 -> /power/VCC5
- C6 pad 1: /VCC1 -> /power/VCC1
- C7 pad 1: /VCC2 -> /power/VCC2
- C8 pad 1: /VCC3 -> /power/VCC3
- C9 pad 1: /VCC4 -> /power/VCC4
- J4 pad A4/B9: /power/VBUS -> /USB interface/VBUS
- J4 pad B4/A9: /power/VBUS -> /USB interface/VBUS
- Q1 pad 2: /VCC5 -> /sensor/VCC5
- R2 pad 1: /VCC1 -> /power/VCC1
- R26 pad 1: /power/VBUS -> /USB interface/VBUS
- R3 pad 1: /VCC2 -> /power/VCC2
- R39 pad 2: PA1 -> /power/REF
- R4 pad 1: /VCC3 -> /power/VCC3
- R40 pad 1: /VCC5 -> /power/VCC5
- R5 pad 1: /VCC4 -> /power/VCC4
- U1 pad 8: /VCC1 -> /sensor/VCC1
- U2 pad 8: /VCC2 -> /sensor/VCC2
- U4 pad 2: /VCC3 -> /sensor/VCC3
- U5 pad 5: /VCC4 -> /sensor/VCC4
- U7 pad 5: /power/VBUS -> /USB interface/VBUS
Routing:
- net /power/VBUS: track 45.3 -> 0.00 mm, vias 4 -> 0
- net /USB interface/VBUS: track 0.00 -> 45.3 mm, vias 0 -> 4
- net /power/VCC5: track 0.00 -> 23.5 mm
- net /VCC5: track 23.5 -> 0.00 mm
- net /power/VCC3: track 0.00 -> 9.36 mm
- net /VCC3: track 9.36 -> 0.00 mm
- net /power/VCC4: track 0.00 -> 6.93 mm
- net /VCC4: track 6.93 -> 0.00 mm
- net /power/VCC2: track 0.00 -> 6.76 mm
- net /VCC2: track 6.76 -> 0.00 mm
- net /power/VCC1: track 0.00 -> 6.63 mm
- net /VCC1: track 6.63 -> 0.00 mm

Commit message: Schematics cleanup of power symbols and routing.
Connections:
- net UAV_5V renamed PixHawk_5V
- J4 pad A4/B9: /USB interface/VBUS -> /USB interface/VUSB
- J4 pad B4/A9: /USB interface/VBUS -> /USB interface/VUSB
- R26 pad 1: /USB interface/VBUS -> /USB interface/VUSB
Routing:
- net /USB interface/VUSB: track 0.00 -> 45.3 mm, vias 0 -> 4
- net /USB interface/VBUS: track 45.3 -> 0.00 mm, vias 4 -> 0
Changed lines of the file:
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@@
   (net 40 "Net-(D3-Pad1)")
   (net 41 "Net-(D4-Pad1)")
-  (net 42 "UAV_5V")
+  (net 42 "PixHawk_5V")
   (net 43 "unconnected-(U10-Pad21)")
   (net 44 "/cpu/TIMEPULSE")
@@
   (net 128 "/sensor/VCC3")
   (net 129 "/sensor/VCC4")
+  (net 130 "/USB interface/VUSB")
   (footprint "Mlab_Mechanical:MountingHole_3mm" placed (layer "F.Cu")
     (at 174.972341 78.676927)
@@
     (fp_line (start -3.125 0.892893) (end -2.625 1.6) (layer "B.Fab") (width 0.1))
     (pad "1" smd roundrect (at -3.125 1.85 270) (size 0.6 1.7) (layers "B.Cu" "B.Paste" "B.Mask") (roundrect_rratio 0.25)
-      (net 42 "UAV_5V") (pintype "input"))
+      (net 42 "PixHawk_5V") (pintype "input"))
     (pad "2" smd roundrect (at -1.875 1.85 270) (size 0.6 1.7) (layers "B.Cu" "B.Paste" "B.Mask") (roundrect_rratio 0.25)
       (net 90 "Net-(J3-Pad2)") (pintype "input"))
@@
       (net 45 "Net-(D5-Pad1)") (pinfunction "K") (pintype "passive"))
     (pad "2" smd rect (at 0.7 0 180) (size 0.6 0.7) (layers "B.Cu" "B.Paste" "B.Mask")
-      (net 42 "UAV_5V") (pinfunction "A") (pintype "passive"))
+      (net 42 "PixHawk_5V") (pinfunction "A") (pintype "passive"))
     (model "${KICAD6_3DMODEL_DIR}/Diode_SMD.3dshapes/D_SOD-523.wrl"
       (offset (xyz 0 0 0))
@@
       (net 1 "GND") (pinfunction "GND") (pintype "passive"))
     (pad "A4/B9" smd rect locked (at -2.4 4.755 270) (size 0.6 1.15) (layers "B.Cu" "B.Paste" "B.Mask")
-      (net 111 "/USB interface/VBUS") (pinfunction "VBUS") (pintype "passive"))
+      (net 130 "/USB interface/VUSB") (pinfunction "VBUS") (pintype "passive"))
     (pad "A5" smd rect locked (at -1.25 4.755 270) (size 0.3 1.15) (layers "B.Cu" "B.Paste" "B.Mask")
       (net 78 "Net-(J4-PadA5)") (pinfunction "CC1") (pintype "bidirectional"))
@@
       (net 1 "GND") (pinfunction "GND") (pintype "passive"))
     (pad "B4/A9" smd rect locked (at 2.4 4.755 270) (size 0.6 1.15) (layers "B.Cu" "B.Paste" "B.Mask")
-      (net 111 "/USB interface/VBUS") (pinfunction "VBUS") (pintype "passive"))
+      (net 130 "/USB interface/VUSB") (pinfunction "VBUS") (pintype "passive"))
     (pad "B5" smd rect locked (at 1.75 4.755 270) (size 0.3 1.15) (layers "B.Cu" "B.Paste" "B.Mask")
       (net 80 "Net-(J4-PadB5)") (pinfunction "CC2") (pintype "bidirectional"))
@@
     (fp_line (start 0.8 -0.4125) (end -0.8 -0.4125) (layer "B.Fab") (width 0.1))
     (pad "1" smd roundrect (at -0.825 0 180) (size 0.8 0.95) (layers "B.Cu" "B.Paste" "B.Mask") (roundrect_rratio 0.25)
-      (net 111 "/USB interface/VBUS") (pintype "passive"))
+      (net 130 "/USB interface/VUSB") (pintype "passive"))
     (pad "2" smd roundrect (at 0.825 0 180) (size 0.8 0.95) (layers "B.Cu" "B.Paste" "B.Mask") (roundrect_rratio 0.25)
       (net 71 "Net-(R26-Pad2)") (pintype "passive"))
@@
   (segment (start 180.663841 118.404427) (end 180.560341 118.300927) (width 0.3) (layer "B.Cu") (net 110))
   (segment (start 182.409341 118.404427) (end 180.663841 118.404427) (width 0.3) (layer "B.Cu") (net 110))
-  (segment (start 180.814341 106.870927) (end 181.576341 106.108927) (width 0.4) (layer "F.Cu") (net 111))
-  (segment (start 181.576341 106.108927) (end 181.576341 97.218927) (width 0.4) (layer "F.Cu") (net 111))
-  (segment (start 180.814341 110.851889) (end 180.85586 110.893408) (width 0.4) (layer "F.Cu") (net 111))
-  (segment (start 180.814341 106.870927) (end 180.814341 110.851889) (width 0.4) (layer "F.Cu") (net 111))
-  (segment (start 171.924341 111.696927) (end 177.323319 111.696927) (width 0.4) (layer "F.Cu") (net 111))
-  (segment (start 177.323319 111.696927) (end 178.12283 110.897416) (width 0.4) (layer "F.Cu") (net 111))
-  (segment (start 180.851852 110.897416) (end 180.85586 110.893408) (width 0.4) (layer "F.Cu") (net 111))
-  (segment (start 180.85586 110.893408) (end 181.359852 111.3974) (width 0.4) (layer "F.Cu") (net 111))
-  (segment (start 178.12283 110.897416) (end 180.851852 110.897416) (width 0.4) (layer "F.Cu") (net 111))
-  (segment (start 181.359852 119.533416) (end 180.814341 120.078927) (width 0.4) (layer "F.Cu") (net 111))
-  (segment (start 181.359852 111.3974) (end 181.359852 119.533416) (width 0.4) (layer "F.Cu") (net 111))
-  (via (at 171.924341 111.696927) (size 0.8) (drill 0.4) (layers "F.Cu" "B.Cu") (net 111))
-  (via (at 180.85586 110.893408) (size 0.8) (drill 0.4) (layers "F.Cu" "B.Cu") (net 111))
-  (via (at 180.814341 120.078927) (size 0.8) (drill 0.4) (layers "F.Cu" "B.Cu") (net 111))
-  (via (at 181.576341 97.218927) (size 0.8) (drill 0.4) (layers "F.Cu" "B.Cu") (net 111))
-  (segment (start 182.409341 115.254427) (end 181.365361 115.254427) (width 0.4) (layer "B.Cu") (net 111))
-  (segment (start 180.855861 114.744927) (end 180.85586 113.516446) (width 0.4) (layer "B.Cu") (net 111))
-  (segment (start 170.717341 111.696927) (end 171.924341 111.696927) (width 0.4) (layer "B.Cu") (net 111))
-  (segment (start 180.85586 112.754446) (end 180.85586 110.893408) (width 0.4) (layer "B.Cu") (net 111))
-  (segment (start 181.576341 96.010927) (end 181.514341 95.948927) (width 0.4) (layer "B.Cu") (net 111))
-  (segment (start 182.384841 120.078927) (end 182.409341 120.054427) (width 0.4) (layer "B.Cu") (net 111))
-  (segment (start 180.814341 112.712927) (end 180.85586 112.754446) (width 0.4) (layer "B.Cu") (net 111))
-  (segment (start 181.576341 97.218927) (end 181.576341 96.010927) (width 0.4) (layer "B.Cu") (net 111))
-  (segment (start 180.052341 112.712927) (end 180.814341 112.712927) (width 0.4) (layer "B.Cu") (net 111))
-  (segment (start 180.052341 112.712927) (end 178.141841 112.712927) (width 0.4) (layer "B.Cu") (net 111))
-  (segment (start 180.814341 120.078927) (end 182.384841 120.078927) (width 0.4) (layer "B.Cu") (net 111))
-  (segment (start 181.365361 115.254427) (end 180.855861 114.744927) (width 0.4) (layer "B.Cu") (net 111))
-  (segment (start 180.85586 113.516446) (end 180.85586 112.754446) (width 0.4) (layer "B.Cu") (net 111))
   (segment (start 168.026341 112.242927) (end 169.726341 112.242927) (width 0.25) (layer "F.Cu") (net 112))
   (segment (start 171.871352 110.097916) (end 174.172841 110.097916) (width 0.25) (layer "F.Cu") (net 112))
@@
   (segment (start 115.828941 88.765327) (end 115.828941 89.611127) (width 0.4) (layer "B.Cu") (net 124))
   (segment (start 115.922341 88.671927) (end 115.828941 88.765327) (width 0.4) (layer "B.Cu") (net 124))
+  (segment (start 180.814341 106.870927) (end 181.576341 106.108927) (width 0.4) (layer "F.Cu") (net 130))
+  (segment (start 181.576341 106.108927) (end 181.576341 97.218927) (width 0.4) (layer "F.Cu") (net 130))
+  (segment (start 180.814341 110.851889) (end 180.85586 110.893408) (width 0.4) (layer "F.Cu") (net 130))
+  (segment (start 180.814341 106.870927) (end 180.814341 110.851889) (width 0.4) (layer "F.Cu") (net 130))
+  (segment (start 171.924341 111.696927) (end 177.323319 111.696927) (width 0.4) (layer "F.Cu") (net 130))
+  (segment (start 177.323319 111.696927) (end 178.12283 110.897416) (width 0.4) (layer "F.Cu") (net 130))
+  (segment (start 180.851852 110.897416) (end 180.85586 110.893408) (width 0.4) (layer "F.Cu") (net 130))
+  (segment (start 180.85586 110.893408) (end 181.359852 111.3974) (width 0.4) (layer "F.Cu") (net 130))
+  (segment (start 178.12283 110.897416) (end 180.851852 110.897416) (width 0.4) (layer "F.Cu") (net 130))
+  (segment (start 181.359852 119.533416) (end 180.814341 120.078927) (width 0.4) (layer "F.Cu") (net 130))
+  (segment (start 181.359852 111.3974) (end 181.359852 119.533416) (width 0.4) (layer "F.Cu") (net 130))
+  (via (at 171.924341 111.696927) (size 0.8) (drill 0.4) (layers "F.Cu" "B.Cu") (net 130))
+  (via (at 180.85586 110.893408) (size 0.8) (drill 0.4) (layers "F.Cu" "B.Cu") (net 130))
+  (via (at 180.814341 120.078927) (size 0.8) (drill 0.4) (layers "F.Cu" "B.Cu") (net 130))
+  (via (at 181.576341 97.218927) (size 0.8) (drill 0.4) (layers "F.Cu" "B.Cu") (net 130))
+  (segment (start 182.409341 115.254427) (end 181.365361 115.254427) (width 0.4) (layer "B.Cu") (net 130))
+  (segment (start 180.855861 114.744927) (end 180.85586 113.516446) (width 0.4) (layer "B.Cu") (net 130))
+  (segment (start 170.717341 111.696927) (end 171.924341 111.696927) (width 0.4) (layer "B.Cu") (net 130))
+  (segment (start 180.85586 112.754446) (end 180.85586 110.893408) (width 0.4) (layer "B.Cu") (net 130))
+  (segment (start 181.576341 96.010927) (end 181.514341 95.948927) (width 0.4) (layer "B.Cu") (net 130))
+  (segment (start 182.384841 120.078927) (end 182.409341 120.054427) (width 0.4) (layer "B.Cu") (net 130))
+  (segment (start 180.814341 112.712927) (end 180.85586 112.754446) (width 0.4) (layer "B.Cu") (net 130))
+  (segment (start 181.576341 97.218927) (end 181.576341 96.010927) (width 0.4) (layer "B.Cu") (net 130))
+  (segment (start 180.052341 112.712927) (end 180.814341 112.712927) (width 0.4) (layer "B.Cu") (net 130))
+  (segment (start 180.052341 112.712927) (end 178.141841 112.712927) (width 0.4) (layer "B.Cu") (net 130))
+  (segment (start 180.814341 120.078927) (end 182.384841 120.078927) (width 0.4) (layer "B.Cu") (net 130))
+  (segment (start 181.365361 115.254427) (end 180.855861 114.744927) (width 0.4) (layer "B.Cu") (net 130))
+  (segment (start 180.85586 113.516446) (end 180.85586 112.754446) (width 0.4) (layer "B.Cu") (net 130))
   (zone (net 1) (net_name "GND") (layers "F.Cu" "In1.Cu" "In2.Cu" "B.Cu") (hatch edge 0.508)
     (connect_pads yes (clearance 0.2))

Commit message: Cleanup schematics Note polarity to ceramic capacitors.
Parts:
- C5: value 1pFNP0 251R15S1R0AV4E -> 1pF/NP0 251R15S1R0AV4E
Connections:
- net +3V3 renamed +3.3V
- C11 pad 1: /power/VCC1 -> /sensor/VCC1
- C12 pad 1: /power/VCC2 -> /sensor/VCC2
- C13 pad 1: /power/VCC3 -> /sensor/VCC3
- C14 pad 1: /power/VCC4 -> /sensor/VCC4
- C53 pad 1: /power/VCC5 -> /sensor/VCC5
- C59 pad 1: /power/VCC5 -> /sensor/VCC5
- C6 pad 1: /power/VCC1 -> /sensor/VCC1
- C7 pad 1: /power/VCC2 -> /sensor/VCC2
- C8 pad 1: /power/VCC3 -> /sensor/VCC3
- C9 pad 1: /power/VCC4 -> /sensor/VCC4
- D5 pad 2: /power/VBUS -> /USB interface/VUSB
- R2 pad 1: /power/VCC1 -> /sensor/VCC1
- R3 pad 1: /power/VCC2 -> /sensor/VCC2
- R39 pad 2: /power/REF -> PA1
- R4 pad 1: /power/VCC3 -> /sensor/VCC3
- R40 pad 1: /power/VCC5 -> /sensor/VCC5
- R5 pad 1: /power/VCC4 -> /sensor/VCC4
- U7 pad 5: /USB interface/VBUS -> /USB interface/VUSB
Routing:
- net /sensor/VCC5: track 0.00 -> 23.5 mm
- net /power/VCC5: track 23.5 -> 0.00 mm
- net /sensor/VCC3: track 0.00 -> 9.36 mm
- net /power/VCC3: track 9.36 -> 0.00 mm
- net /sensor/VCC4: track 0.00 -> 6.93 mm
- net /power/VCC4: track 6.93 -> 0.00 mm
- net /sensor/VCC2: track 0.00 -> 6.76 mm
- net /power/VCC2: track 6.76 -> 0.00 mm
- net /sensor/VCC1: track 0.00 -> 6.63 mm
- net /power/VCC1: track 6.63 -> 0.00 mm

Commit message: Add notes to schematics.
Connections:
- C17 pad 1: PA1 -> /sensor/REF
- C24 pad 2: PA1 -> /sensor/REF
- C3 pad 1: PA1 -> /sensor/REF
- R39 pad 2: PA1 -> /sensor/REF
- R7 pad 1: PA1 -> /sensor/REF
- R8 pad 2: PA1 -> /sensor/REF
- U1 pad 3: PA1 -> /sensor/REF
- U10 pad 36: PA1 -> /cpu/Voltage_Reference
- U2 pad 3: PA1 -> /sensor/REF
Routing:
- net PA1: track 107.5 -> 0.00 mm, vias 3 -> 0
- net /sensor/REF: track 0.00 -> 107.5 mm, vias 0 -> 3
Changed lines of the file:
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@@
   (net 28 "+5V")
   (net 29 "Net-(L3-Pad2)")
-  (net 30 "PA1")
+  (net 30 "/sensor/REF")
   (net 31 "PA0")
   (net 32 "Net-(C40-Pad1)")
@@
   (net 121 "/sensor/VCC4")
   (net 122 "/USB interface/VUSB")
+  (net 123 "/cpu/Voltage_Reference")
   (footprint "Mlab_Mechanical:MountingHole_3mm" placed (layer "F.Cu")
     (at 174.972341 78.676927)
@@
     (fp_line (start 0.8 0.4) (end 0.8 -0.4) (layer "B.Fab") (width 0.1))
     (pad "1" smd roundrect (at -0.775 0 90) (size 0.9 0.95) (layers "B.Cu" "B.Paste" "B.Mask") (roundrect_rratio 0.25)
-      (net 30 "PA1") (pintype "passive"))
+      (net 30 "/sensor/REF") (pintype "passive"))
     (pad "2" smd roundrect (at 0.775 0 90) (size 0.9 0.95) (layers "B.Cu" "B.Paste" "B.Mask") (roundrect_rratio 0.25)
       (net 1 "GND") (pintype "passive"))
@@
     (fp_line (start 0.8 -0.4) (end -0.8 -0.4) (layer "B.Fab") (width 0.1))
     (pad "1" smd roundrect (at -0.775 0 180) (size 0.9 0.95) (layers "B.Cu" "B.Paste" "B.Mask") (roundrect_rratio 0.25)
-      (net 30 "PA1") (pintype "passive"))
+      (net 30 "/sensor/REF") (pintype "passive"))
     (pad "2" smd roundrect (at 0.775 0 180) (size 0.9 0.95) (layers "B.Cu" "B.Paste" "B.Mask") (roundrect_rratio 0.25)
       (net 1 "GND") (pintype "passive"))
@@
     (fp_line (start 0.8 -0.4125) (end -0.8 -0.4125) (layer "B.Fab") (width 0.1))
     (pad "1" smd roundrect (at -0.825 0 270) (size 0.8 0.95) (layers "B.Cu" "B.Paste" "B.Mask") (roundrect_rratio 0.25)
-      (net 30 "PA1") (pintype "passive"))
+      (net 30 "/sensor/REF") (pintype "passive"))
     (pad "2" smd roundrect (at 0.825 0 270) (size 0.8 0.95) (layers "B.Cu" "B.Paste" "B.Mask") (roundrect_rratio 0.25)
       (net 3 "Net-(C10-Pad1)") (pintype "passive"))
@@
       (net 5 "Net-(C15-Pad2)") (pintype "passive"))
     (pad "2" smd roundrect (at 0.825 0 90) (size 0.8 0.95) (layers "B.Cu" "B.Paste" "B.Mask") (roundrect_rratio 0.25)
-      (net 30 "PA1") (pintype "passive"))
+      (net 30 "/sensor/REF") (pintype "passive"))
     (model "${KICAD6_3DMODEL_DIR}/Resistor_SMD.3dshapes/R_0603_1608Metric.wrl"
       (offset (xyz 0 0 0))
@@
       (net 114 "/sensor/A") (pinfunction "-") (pintype "input"))
     (pad "3" smd roundrect (at -2.475 -0.635) (size 1.95 0.6) (layers "B.Cu" "B.Paste" "B.Mask") (roundrect_rratio 0.25)
-      (net 30 "PA1") (pinfunction "+") (pintype "input"))
+      (net 30 "/sensor/REF") (pinfunction "+") (pintype "input"))
     (pad "4" smd roundrect (at -2.475 -1.905) (size 1.95 0.6) (layers "B.Cu" "B.Paste" "B.Mask") (roundrect_rratio 0.25)
       (net 1 "GND") (pinfunction "V-") (pintype "power_in"))
@@
       (net 8 "Net-(C18-Pad2)") (pinfunction "-") (pintype "input"))
     (pad "3" smd roundrect (at -2.475 -0.635) (size 1.95 0.6) (layers "B.Cu" "B.Paste" "B.Mask") (roundrect_rratio 0.25)
-      (net 30 "PA1") (pinfunction "+") (pintype "input"))
+      (net 30 "/sensor/REF") (pinfunction "+") (pintype "input"))
     (pad "4" smd roundrect (at -2.475 -1.905) (size 1.95 0.6) (layers "B.Cu" "B.Paste" "B.Mask") (roundrect_rratio 0.25)
       (net 1 "GND") (pinfunction "V-") (pintype "power_in"))
@@
       (net 52 "unconnected-(U10-Pad35)") (pinfunction "(PCINT2/ADC2)PA2") (pintype "bidirectional+no_connect"))
     (pad "36" smd rect (at 2.4 5.7 270) (size 1.5 0.55) (layers "B.Cu" "B.Paste" "B.Mask")
-      (net 30 "PA1") (pinfunction "(PCINT1/ADC1)PA1") (pintype "bidirectional"))
+      (net 123 "/cpu/Voltage_Reference") (pinfunction "(PCINT1/ADC1)PA1") (pintype "bidirectional"))
     (pad "37" smd rect (at 1.6 5.7 270) (size 1.5 0.55) (layers "B.Cu" "B.Paste" "B.Mask")
       (net 31 "PA0") (pinfunction "(PCINT0/ADC0)PA0") (pintype "bidirectional"))
@@
       (net 115 "/sensor/Ubiasout") (pintype "passive"))
     (pad "2" smd roundrect (at 0.775 0 270) (size 0.9 0.95) (layers "B.Cu" "B.Paste" "B.Mask") (roundrect_rratio 0.25)
-      (net 30 "PA1") (pintype "passive"))
+      (net 30 "/sensor/REF") (pintype "passive"))
     (model "${KICAD6_3DMODEL_DIR}/Capacitor_SMD.3dshapes/C_0603_1608Metric.wrl"
       (offset (xyz 0 0 0))
@@
       (net 96 "Net-(C20-Pad1)") (pintype "passive"))
     (pad "2" smd roundrect (at 0.825 0 180) (size 0.8 0.95) (layers "B.Cu" "B.Paste" "B.Mask") (roundrect_rratio 0.25)
-      (net 30 "PA1") (pintype "passive"))
+      (net 30 "/sensor/REF") (pintype "passive"))
     (model "${KICAD6_3DMODEL_DIR}/Resistor_SMD.3dshapes/R_0603_1608Metric.wrl"
       (offset (xyz 0 0 0))

Commit message: Changed voltage reference to 0.9V.
Parts:
- U3: value ISL21080DIH312Z-TK 1V25 -> ISL21080DIH309ZT
Connections:
- U10 pad 36: /cpu/Voltage_Reference -> /sensor/REF
Changed lines of the file:
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@@
   (net 121 "/sensor/VCC4")
   (net 122 "/USB interface/VUSB")
-  (net 123 "/cpu/Voltage_Reference")
   (footprint "Mlab_Mechanical:MountingHole_3mm" placed (layer "F.Cu")
     (at 174.972341 78.676927)
@@
     (property "Sheetfile" "power.kicad_sch")
     (property "Sheetname" "power")
-    (property "UST_ID" "5c70984712875079b91f8b7a")
+    (property "UST_ID" "5c70984712875079b91f8b0b")
     (attr smd)
     (fp_text reference "U3" (at 1.304 -1.742 180) (layer "B.SilkS")
       (effects (font (size 1 1) (thickness 0.15)) (justify mirror))
     )
-    (fp_text value "ISL21080DIH312Z-TK  1V25" (at 0 -2.5 90) (layer "B.Fab") hide
+    (fp_text value "ISL21080DIH309ZT" (at 0 -2.5 90) (layer "B.Fab") hide
       (effects (font (size 1 1) (thickness 0.15)) (justify mirror))
     )
@@
       (net 52 "unconnected-(U10-Pad35)") (pinfunction "(PCINT2/ADC2)PA2") (pintype "bidirectional+no_connect"))
     (pad "36" smd rect (at 2.4 5.7 270) (size 1.5 0.55) (layers "B.Cu" "B.Paste" "B.Mask")
-      (net 123 "/cpu/Voltage_Reference") (pinfunction "(PCINT1/ADC1)PA1") (pintype "bidirectional"))
+      (net 30 "/sensor/REF") (pinfunction "(PCINT1/ADC1)PA1") (pintype "bidirectional"))
     (pad "37" smd rect (at 1.6 5.7 270) (size 1.5 0.55) (layers "B.Cu" "B.Paste" "B.Mask")
       (net 31 "PA0") (pinfunction "(PCINT0/ADC0)PA0") (pintype "bidirectional"))
