File: hw/sch_pcb/USTSIPIN02A.kicad_pcb (KiCad board)
At the start: 4 copper layers, 90.9 x 50.3 mm, 154 parts, among them J1 SM08B-GHS-TB, J2 SD_Card-FPS009-4200-0, J22 HEADER_2x03, J3 SM06B-GHS-TB, J4 USBC_USB4105-GF-A, J5 HEADER_1x01, J6 HEADER_1x01, J7 SM03B-GHS-TB, M1 HOLE, M2 HOLE, M3 HOLE, M4 HOLE, M8 BMI-S-204-F, Q1 2SK2394-6, Q2 BC817-25, Q3 BC817-25, Q4 BC817-25, U1 OPA2314, U10 ATMEGA1284P-AU, U11 PCF85263A, U12 MIC5504-3.3YM5, U2 OPA2314, U3 ISL21080DIH309ZT, U4 TS7211, U5 TS5A4594, U6 AT24CS64-SSHM, U7 USBLC6-2SC6, U8 TPS613222ADBV, U9 FT231XQ, Y1 8 MHz, Y2 ABS07-120-32.768KHZ-T

Commit message: swapping 100nF and 10uF
Parts:
- C11, C13: value 100nF -> 10uF
- C6, C8: value 10uF -> 100nF
- R2, R4, R40, R5: value 470R -> 100R
- R3: value 10R -> 100R
- U12: value MIC5504-3.3YM5 -> LP2985AIM5-3.6
Changed lines of the file:
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@@
     (property "Sheetfile" "power.kicad_sch")
     (property "Sheetname" "power")
-    (property "UST_ID" "5c70984812875079b91f8bf5")
+    (property "UST_ID" "643f075476c82a1d3b576c19")
     (attr smd)
     (fp_text reference "C1" (at -2.4244 -0.0612) (layer "B.SilkS")
@@
     (property "Sheetfile" "sensor.kicad_sch")
     (property "Sheetname" "sensor")
-    (property "UST_ID" "5c70984812875079b91f8bc2")
+    (property "UST_ID" "643f03ef76c82a1d3b576bed")
     (attr smd)
     (fp_text reference "C3" (at 0.5975 -1.29 270) (layer "B.SilkS")
@@
     (property "Sheetfile" "power.kicad_sch")
     (property "Sheetname" "power")
-    (property "UST_ID" "5c70984812875079b91f8bf5")
+    (property "UST_ID" "643f075476c82a1d3b576c19")
     (attr smd)
     (fp_text reference "C4" (at -2.3244 -0.0316) (layer "B.SilkS")
@@
     (property "Sheetfile" "sensor.kicad_sch")
     (property "Sheetname" "sensor")
-    (property "UST_ID" "5c70984812875079b91f8bf5")
+    (property "UST_ID" "5c70984812875079b91f8bf2")
     (attr smd)
     (fp_text reference "C6" (at 0 1.43 90) (layer "B.SilkS")
       (effects (font (size 1 1) (thickness 0.15)) (justify mirror))
     )
-    (fp_text value "10uF" (at 0 -1.43 90) (layer "B.Fab") hide
+    (fp_text value "100nF" (at 0 -1.43 90) (layer "B.Fab") hide
       (effects (font (size 1 1) (thickness 0.15)) (justify mirror))
     )
@@
     (property "Sheetfile" "sensor.kicad_sch")
     (property "Sheetname" "sensor")
-    (property "UST_ID" "5c70984812875079b91f8bf5")
+    (property "UST_ID" "643f075476c82a1d3b576c19")
     (attr smd)
     (fp_text reference "C7" (at -2.1128 -0.162 90) (layer "B.SilkS")
@@
     (property "Sheetfile" "sensor.kicad_sch")
     (property "Sheetname" "sensor")
-    (property "UST_ID" "5c70984812875079b91f8bf5")
+    (property "UST_ID" "")
     (attr smd)
     (fp_text reference "C8" (at -1.9492 0.0236 90) (layer "B.SilkS")
       (effects (font (size 0.8 0.8) (thickness 0.1)) (justify mirror))
     )
-    (fp_text value "10uF" (at 0 -1.43) (layer "B.Fab") hide
+    (fp_text value "100nF" (at 0 -1.43) (layer "B.Fab") hide
       (effects (font (size 1 1) (thickness 0.15)) (justify mirror))
     )
@@
     (property "Sheetfile" "sensor.kicad_sch")
     (property "Sheetname" "sensor")
-    (property "UST_ID" "5c70984812875079b91f8bf5")
+    (property "UST_ID" "643f075476c82a1d3b576c19")
     (attr smd)
     (fp_text reference "C9" (at 0 1.43) (layer "B.SilkS")
@@
     (property "Sheetfile" "sensor.kicad_sch")
     (property "Sheetname" "sensor")
-    (property "UST_ID" "5c70984812875079b91f8bf2")
+    (property "UST_ID" "643f075476c82a1d3b576c19")
     (attr smd)
     (fp_text reference "C11" (at 0 1.43 90) (layer "B.SilkS") hide
       (effects (font (size 1 1) (thickness 0.15)) (justify mirror))
     )
-    (fp_text value "100nF" (at 0 -1.43 90) (layer "B.Fab") hide
+    (fp_text value "10uF" (at 0 -1.43 90) (layer "B.Fab") hide
       (effects (font (size 1 1) (thickness 0.15)) (justify mirror))
     )
@@
     (property "Sheetfile" "sensor.kicad_sch")
     (property "Sheetname" "sensor")
-    (property "UST_ID" "5c70984812875079b91f8bf2")
+    (property "UST_ID" "")
     (attr smd)
     (fp_text reference "C13" (at 0.8508 1.0956) (layer "B.SilkS")
       (effects (font (size 0.8 0.8) (thickness 0.1)) (justify mirror))
     )
-    (fp_text value "100nF" (at 0 -1.43) (layer "B.Fab") hide
+    (fp_text value "10uF" (at 0 -1.43) (layer "B.Fab") hide
       (effects (font (size 1 1) (thickness 0.15)) (justify mirror))
     )
@@
     (property "Sheetfile" "sensor.kicad_sch")
     (property "Sheetname" "sensor")
-    (property "UST_ID" "5c70984812875079b91f8bc2")
+    (property "UST_ID" "643f03ef76c82a1d3b576bed")
     (attr smd)
     (fp_text reference "C17" (at 0 1.43) (layer "B.SilkS")
@@
     (property "Sheetfile" "sensor.kicad_sch")
     (property "Sheetname" "sensor")
-    (property "UST_ID" "5c70984512875079b91f894f")
+    (property "UST_ID" "5c70984512875079b91f8956")
     (attr smd)
     (fp_text reference "R3" (at -0.1312 -1.4024 90) (layer "B.SilkS")
       (effects (font (size 1 1) (thickness 0.15)) (justify mirror))
     )
-    (fp_text value "10R" (at 0 -1.43 90) (layer "B.Fab") hide
+    (fp_text value "100R" (at 0 -1.43 90) (layer "B.Fab") hide
       (effects (font (size 1 1) (thickness 0.15)) (justify mirror))
     )
@@
     (property "Sheetfile" "sensor.kicad_sch")
     (property "Sheetname" "sensor")
-    (property "UST_ID" "5c70984512875079b91f8959")
+    (property "UST_ID" "5c70984512875079b91f8956")
     (attr smd)
     (fp_text reference "R4" (at -2.0492 0.0524 90) (layer "B.SilkS")
       (effects (font (size 0.8 0.8) (thickness 0.1)) (justify mirror))
     )
-    (fp_text value "470R" (at 0 -1.43) (layer "B.Fab") hide
+    (fp_text value "100R" (at 0 -1.43) (layer "B.Fab") hide
       (effects (font (size 1 1) (thickness 0.15)) (justify mirror))
     )
@@
     (property "Sheetfile" "sensor.kicad_sch")
     (property "Sheetname" "sensor")
-    (property "UST_ID" "5c70984512875079b91f8959")
+    (property "UST_ID" "5c70984512875079b91f8956")
     (attr smd)
     (fp_text reference "R5" (at -0.0256 -1.4296) (layer "B.SilkS")
       (effects (font (size 1 1) (thickness 0.15)) (justify mirror))
     )
-    (fp_text value "470R" (at 0 -1.43) (layer "B.Fab") hide
+    (fp_text value "100R" (at 0 -1.43) (layer "B.Fab") hide
       (effects (font (size 1 1) (thickness 0.15)) (justify mirror))
     )
@@
     (property "Sheetfile" "sensor.kicad_sch")
     (property "Sheetname" "sensor")
-    (property "UST_ID" "5c70984512875079b91f8959")
+    (property "UST_ID" "5c70984512875079b91f8956")
     (attr smd)
     (fp_text reference "R2" (at 0 1.43 90) (layer "B.SilkS") hide
       (effects (font (size 1 1) (thickness 0.15)) (justify mirror))
     )
-    (fp_text value "470R" (at 0 -1.43 90) (layer "B.Fab") hide
+    (fp_text value "100R" (at 0 -1.43 90) (layer "B.Fab") hide
       (effects (font (size 1 1) (thickness 0.15)) (justify mirror))
     )
@@
     (property "Sheetfile" "sensor.kicad_sch")
     (property "Sheetname" "sensor")
-    (property "UST_ID" "5c70984812875079b91f8bf5")
+    (property "UST_ID" "643f075476c82a1d3b576c19")
     (attr smd)
     (fp_text reference "C21" (at -0.0068 -1.472 90) (layer "B.SilkS")
@@
     (property "Sheetfile" "power.kicad_sch")
     (property "Sheetname" "power")
-    (property "UST_ID" "5c70984812875079b91f8bf5")
+    (property "UST_ID" "643f075476c82a1d3b576c19")
     (attr smd)
     (fp_text reference "C50" (at 1.105 1.488 270) (layer "B.SilkS")
@@
     (property "Sheetfile" "power.kicad_sch")
     (property "Sheetname" "power")
-    (property "UST_ID" "5c70984812875079b91f8bf5")
+    (property "UST_ID" "643f075476c82a1d3b576c19")
     (attr smd)
     (fp_text reference "C42" (at 1.805 -1.48 90) (layer "B.SilkS")
@@
     (property "Sheetfile" "sensor.kicad_sch")
     (property "Sheetname" "sensor")
-    (property "UST_ID" "5c70984812875079b91f8bf5")
+    (property "UST_ID" "643f075476c82a1d3b576c19")
     (attr smd)
     (fp_text reference "C23" (at 2.9432 -0.1056 90) (layer "B.SilkS")
@@
     (property "Sheetfile" "sensor.kicad_sch")
     (property "Sheetname" "sensor")
-    (property "UST_ID" "5c70984812875079b91f8bc2")
+    (property "UST_ID" "643f03ef76c82a1d3b576bed")
     (attr smd)
     (fp_text reference "C24" (at 0 1.43 90) (layer "B.SilkS") hide
@@
     (property "Sheetfile" "power.kicad_sch")
     (property "Sheetname" "power")
-    (property "UST_ID" "5c70984812875079b91f8bf5")
+    (property "UST_ID" "643f075476c82a1d3b576c19")
     (attr smd)
     (fp_text reference "C58" (at -0.0276 -1.4296) (layer "B.SilkS")
@@
     (property "Sheetfile" "sensor.kicad_sch")
     (property "Sheetname" "sensor")
-    (property "UST_ID" "5c70984812875079b91f8bc2")
+    (property "UST_ID" "643f03ef76c82a1d3b576bed")
     (attr smd)
     (fp_text reference "C37" (at 0 1.43 90) (layer "B.SilkS") hide
@@
     (property "Sheetfile" "power.kicad_sch")
     (property "Sheetname" "power")
-    (property "UST_ID" "5c70984812875079b91f8bf5")
+    (property "UST_ID" "643f075476c82a1d3b576c19")
     (attr smd)
     (fp_text reference "C55" (at -2.8244 0.2092) (layer "B.SilkS")
@@
     (property "Sheetfile" "power.kicad_sch")
     (property "Sheetname" "power")
-    (property "UST_ID" "5c70984812875079b91f8bf5")
+    (property "UST_ID" "643f075476c82a1d3b576c19")
     (attr smd)
     (fp_text reference "C57" (at -1.0572 -1.346 90) (layer "B.SilkS")
@@
     (property "Sheetfile" "sensor.kicad_sch")
     (property "Sheetname" "sensor")
-    (property "UST_ID" "5c70984512875079b91f8959")
+    (property "UST_ID" "5c70984512875079b91f8956")
     (attr smd)
     (fp_text reference "R40" (at 0.0864 -1.5088 90) (layer "B.SilkS")
       (effects (font (size 1 1) (thickness 0.15)) (justify mirror))
     )
-    (fp_text value "470R" (at 0 -1.43 90) (layer "B.Fab") hide
+    (fp_text value "100R" (at 0 -1.43 90) (layer "B.Fab") hide
       (effects (font (size 1 1) (thickness 0.15)) (justify mirror))
     )
@@
     (property "Sheetfile" "power.kicad_sch")
     (property "Sheetname" "power")
-    (property "UST_ID" "5c70984812875079b91f8bf5")
+    (property "UST_ID" "643f075476c82a1d3b576c19")
     (attr smd)
     (fp_text reference "C56" (at 0.0928 1.2252 90) (layer "B.SilkS")
@@
     (property "Sheetfile" "sensor.kicad_sch")
     (property "Sheetname" "sensor")
-    (property "UST_ID" "5c70984812875079b91f8bf5")
+    (property "UST_ID" "643f075476c82a1d3b576c19")
     (attr smd)
     (fp_text reference "C53" (at -0.902 -2.3876 180) (layer "B.SilkS")
@@
       (effects (font (size 0.8 0.8) (thickness 0.1)) (justify mirror))
     )
-    (fp_text value "MIC5504-3.3YM5" (at 0 -2.4) (layer "B.Fab") hide
+    (fp_text value "LP2985AIM5-3.6" (at 0 -2.4) (layer "B.Fab") hide
       (effects (font (size 1 1) (thickness 0.15)) (justify mirror))
     )

Commit message: Update PCB from schematics.
Parts:
- C13: value 10uF -> 100nF
- C8: value 100nF -> 10uF
Changed lines of the file:
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@@
     (property "Sheetfile" "sensor.kicad_sch")
     (property "Sheetname" "sensor")
-    (property "UST_ID" "")
+    (property "UST_ID" "643f075476c82a1d3b576c19")
     (attr smd)
     (fp_text reference "C8" (at -1.9492 0.0236 90) (layer "B.SilkS")
       (effects (font (size 0.8 0.8) (thickness 0.1)) (justify mirror))
     )
-    (fp_text value "100nF" (at 0 -1.43) (layer "B.Fab") hide
+    (fp_text value "10uF" (at 0 -1.43) (layer "B.Fab") hide
       (effects (font (size 1 1) (thickness 0.15)) (justify mirror))
     )
@@
     (property "Sheetfile" "sensor.kicad_sch")
     (property "Sheetname" "sensor")
-    (property "UST_ID" "")
+    (property "UST_ID" "5c70984812875079b91f8bf2")
     (attr smd)
     (fp_text reference "C13" (at 0.8508 1.0956) (layer "B.SilkS")
       (effects (font (size 0.8 0.8) (thickness 0.1)) (justify mirror))
     )
-    (fp_text value "10uF" (at 0 -1.43) (layer "B.Fab") hide
+    (fp_text value "100nF" (at 0 -1.43) (layer "B.Fab") hide
       (effects (font (size 1 1) (thickness 0.15)) (justify mirror))
     )
